File: ErgoNexus.kicad_pcb (KiCad board)
At the start: 2 copper layers, 132 parts, among them J10 Conn_01x05, J7 Conn_01x02, J8 Conn_01x02, J9 Conn_01x05, SW1 SW_Push, SW2 RotaryEncoder_Switch, SW3 SW_Push, SW4 RotaryEncoder_Switch, U1 SuperMini nRF52840, U2 SuperMini nRF52840

Commit message: feat: 右手のレイアウトを設定
Parts:
- removed D48: 1N4148, kbd_Parts:Diode_TH_SMD
- removed RC0-1, RC0-5, RC1-2, RC1-6, RC2-3, RC3-4, RC6-8: SW_Push, kbd_SW:CherryMX_Hotswap_1u_Small1
- added RC0-7: SW_Push, kbd_SW:CherryMX_Hotswap_1u, F.Cu at (271.9, 132.7)
- added RC0-8: SW_Push, kbd_SW:CherryMX_Hotswap_1u, F.Cu at (244.7, 184.1)
- added RC1-7: SW_Push, kbd_SW:CherryMX_Hotswap_1u, F.Cu at (288.4, 121.6)
- added RC1-8: SW_Push, kbd_SW:CherryMX_Hotswap_1u, F.Cu at (257.0, 166.6)
- added RC2-8: SW_Push, kbd_SW:CherryMX_Hotswap_1u, F.Cu at (275.2, 153.7)
- added RC3-7: SW_Push, kbd_SW:CherryMX_Hotswap_1u, F.Cu at (306.1, 113.6)
- C1, C2, C3, C4: footprint kbd_Parts:Capacitor_1206 -> Capacitor_THT:C_Disc_D3.8mm_W2.6mm_P2.50mm
- J10, J9: value Conn_01x05 -> Conn_01x06; footprint Connector_PinHeader_2.54mm:PinHeader_1x05_P2.54mm_Horizontal -> Connector_PinHeader_2.54mm:PinHeader_1x06_P2.54mm_Horizontal
- J7: moved to B.Cu
- OL7, OL8: footprint Connector_PinSocket_2.54mm:PinSocket_1x04_P2.54mm_Vertical -> kbd_Parts:OLED
- R1, R2, R3, R4: footprint kbd:R -> Keebio-Parts.pretty-master:Resistor-Compact-1-side
- RC0-2, RC0-3, RC0-4, RC0-6, RC1-1, RC1-3, RC1-4, RC1-5, RC2-1, RC2-2, RC2-4, RC2-5, RC2-6, RC3-1, RC3-2, RC3-3, RC3-5, RC3-6, RC4-1, RC4-2, RC4-3, RC4-4, RC4-5, RC4-6, RC4-7, RC4-8, RC5-1, RC5-2, RC5-3, RC5-4, RC5-5, RC5-6, RC5-7, RC5-8, RC6-1, RC6-2, RC6-3, RC6-4, RC6-5, RC6-6, RC6-7: footprint kbd_SW:CherryMX_Hotswap_1u_Small1 -> kbd_SW:CherryMX_Hotswap_1u
- moved RC0-4 141.8 mm to (90.9, 113.1), turned to 14 degrees
- moved RC1-4 117.7 mm to (158.6, 30.0), turned to 7.1 degrees
- moved DI5 116.3 mm to (334.8, 130.6), turned to -160 degrees
- moved DS7 116.1 mm to (324.8, 140.8), turned to -160 degrees
- moved RC0-6 112.3 mm to (265.8, 113.4), turned to 14 degrees
- moved DS6 110.6 mm to (324.8, 137.7), turned to -160 degrees
- moved RC2-6 109.3 mm to (283.1, 102.0), turned to 11.4 degrees
- moved C3 106.3 mm to (295.9, 173.6)
- moved DS5 105.9 mm to (324.6, 134.3), turned to -160 degrees
- moved C4 105.2 mm to (295.8, 181.0)
- moved RC2-4 103.8 mm to (160.2, 76.3), turned to 5 degrees
- moved R3 101.1 mm to (294.4, 167.4)
- moved R4 93.6 mm to (294.4, 186.0)
- moved OL8 82.1 mm to (229.9, 73.6), turned to -82.22 degrees
- moved RC3-6 82.0 mm to (301.1, 93.6), turned to 10 degrees
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Connections:
- net KeyL3 renamed Key3_L
- net KeyL4 renamed Key4_L
- net KeyL5 renamed Key5_L
- net KeyL6 renamed Key6_L
- DS1 pad 1: KeyL0 -> Key0_L
- DS2 pad 1: KeyL1 -> Key1_L
- DS3 pad 1: KeyL2 -> Key2_L
- J10 pad 4: EXT_VCC_R -> CS_R
- J10 pad 5: GND_R -> EXT_VCC_R
- J9 pad 4: EXT_VCC_L -> CS_L
- J9 pad 5: GND_L -> EXT_VCC_L
- RC0-2 pad 1: KeyL0 -> Key0_L
- RC0-2 pad 2: Net-(D2-A) -> Net-(D1-A)
- RC0-3 pad 1: KeyL0 -> Key0_L
- RC0-3 pad 2: Net-(D3-A) -> Net-(D2-A)
- RC0-4 pad 1: Key0_R -> Key0_L
- RC0-4 pad 2: Net-(D25-A) -> Net-(D3-A)
- RC0-6 pad 2: Net-(D27-A) -> Net-(D25-A)
- RC1-1 pad 1: KeyL1 -> Key1_L
- RC1-3 pad 1: KeyL1 -> Key1_L
- RC1-3 pad 2: Net-(D6-A) -> Net-(D5-A)
- RC1-4 pad 1: Key1_R -> Key1_L
- RC1-4 pad 2: Net-(D28-A) -> Net-(D6-A)
- RC1-5 pad 2: Net-(D29-A) -> Net-(D28-A)
- RC2-1 pad 1: KeyL2 -> Key2_L
- RC2-2 pad 1: KeyL2 -> Key2_L
- RC2-4 pad 1: Key2_R -> Key2_L
- RC2-4 pad 2: Net-(D31-A) -> Net-(D9-A)
- RC2-5 pad 2: Net-(D32-A) -> Net-(D31-A)
- RC2-6 pad 2: Net-(D33-A) -> Net-(D32-A)
- RC3-5 pad 2: Net-(D35-A) -> Net-(D34-A)
- RC3-6 pad 2: Net-(D36-A) -> Net-(D35-A)
- U1 pad 10: Ro_B_L -> RoSW_L
- U1 pad 11: unconnected-(U1-P1.04-LF-Pad11) -> Ro_A_L
- U1 pad 12: unconnected-(U1-P1.06-LF-Pad12) -> Ro_B_L
- U1 pad 17: KeyL0 -> Key0_L
- U1 pad 18: KeyL1 -> Key1_L
- U1 pad 19: KeyL2 -> Key2_L
- U1 pad 8: RoSW_L -> CS_L
- U1 pad 9: Ro_A_L -> unconnected-(U1-P1.00-Pad9)
- U2 pad 10: Ro_B_R -> RoSW_R
- U2 pad 11: unconnected-(U2-P1.04-LF-Pad11) -> Ro_A_R
- U2 pad 12: unconnected-(U2-P1.06-LF-Pad12) -> Ro_B_R
- U2 pad 8: RoSW_R -> CS_R
- U2 pad 9: Ro_A_R -> unconnected-(U2-P1.00-Pad9)
Other:
- board outline added: 185.4 x 144.3 mm

Commit message: chore: remove Cuts
Other:
- board outline removed

Commit message: fix: 右手の配線を完成
Parts:
- removed J10: Conn_01x06, Connector_PinHeader_2.54mm:PinHeader_1x06_P2.54mm_Horizontal
- moved DS5 89.7 mm to (235.0, 129.3), turned to 180 degrees
- moved DS6 87.8 mm to (237.1, 132.6), turned to 180 degrees
- moved DS7 85.9 mm to (239.1, 135.7), turned to 180 degrees
- moved DS8 84.0 mm to (240.9, 138.8), turned to 180 degrees
- moved DI5 83.6 mm to (251.3, 127.4), turned to 180 degrees
- moved DI6 83.6 mm to (251.3, 130.6), turned to 180 degrees
- moved DI7 83.6 mm to (251.3, 133.9), turned to 180 degrees
- moved DI8 83.6 mm to (251.3, 136.9), turned to 180 degrees
- moved SW2 64.5 mm to (139.2, 146.0)
- moved SW4 59.8 mm to (333.2, 142.6), turned to 28 degrees
- moved R4 40.1 mm to (321.5, 156.5), turned to -152 degrees
- moved C4 39.6 mm to (323.3, 152.5), turned to 118 degrees
- moved C3 36.1 mm to (321.0, 147.6), turned to 118 degrees
- moved SW3 30.5 mm to (232.7, 123.8), turned to 0 degrees
- moved R3 29.9 mm to (314.4, 145.2), turned to -152 degrees
Routing:
- net Net-(D27-K): track 0.00 -> 231.5 mm, vias 0 -> 2
- net Key5_R: track 0.00 -> 210.1 mm, vias 0 -> 6
- net Net-(D26-K): track 0.00 -> 181.0 mm
- net Net-(D28-K): track 0.00 -> 178.4 mm, vias 0 -> 3
- net Net-(D25-K): track 0.00 -> 173.6 mm
- net Key4_R: track 0.00 -> 162.4 mm, vias 0 -> 3
- net Key6_R: track 0.00 -> 161.6 mm, vias 0 -> 2
- net RoSW_R: track 0.00 -> 158.8 mm, vias 0 -> 1
- net Ro_A_R: track 0.00 -> 146.9 mm
- net Key1_R: track 0.00 -> 134.3 mm, vias 0 -> 2
- net Key0_R: track 0.00 -> 132.1 mm, vias 0 -> 4
- net Key3_R: track 0.00 -> 124.5 mm, vias 0 -> 1
- net Ro_B_R: track 0.00 -> 123.1 mm
- net GND_R: track 0.00 -> 119.7 mm
- net Key2_R: track 0.00 -> 117.4 mm, vias 0 -> 1
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Other:
- board outline added: 174.3 x 138 mm

Commit message: feat: PCBにおいてアノテーションを対応付け
Parts:
- renumbered D28 to D11_R, D31 to D12_R, D34 to D13_R, D37 to D14_R, D25 to D21_R, D32 to D22_R, D35 to D23_R, D38 to D24_R, D41 to D25_R, D45 to D26_R, D26 to D31_R, D29 to D32_R, D36 to D33_R, D39 to D34_R, D42 to D35_R, D46 to D36_R, D44 to D37_R, D27 to D41_R, D30 to D42_R, D33 to D43_R, D40 to D44_R, D43 to D45_R, D47 to D46_R, RC1-5 to K11_R, RC2-5 to K12_R, RC3-5 to K13_R, RC4-5 to K14_R, RC0-6 to K21_R, RC2-6 to K22_R, RC3-6 to K23_R, RC4-6 to K24_R, RC5-5 to K25_R, RC6-5 to K26_R, RC0-7 to K31_R, RC1-7 to K32_R, RC3-7 to K33_R, RC4-7 to K34_R, RC5-6 to K35_R, RC6-6 to K36_R, RC5-8 to K37_R, RC0-8 to K41_R, RC1-8 to K42_R, RC2-8 to K43_R, RC4-8 to K44_R, RC5-7 to K45_R, RC6-7 to K46_R
Changed lines of the file:
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@@
 		(descr "Resitance 3 pas")
 		(tags "R")
-		(property "Reference" "D27"
+		(property "Reference" "D41_R"
 			(at 0 -1.630001 62)
 			(layer "B.SilkS")
@@
 		(descr "Resitance 3 pas")
 		(tags "R")
-		(property "Reference" "D28"
+		(property "Reference" "D11_R"
 			(at 0 -1.63 7.12)
 			(layer "B.SilkS")
@@
 		(layer "F.Cu")
 		(at 280.168077 82.116978 5)
-		(property "Reference" "RC2-5"
+		(property "Reference" "K12_R"
 			(at 0 4 5)
 			(layer "B.SilkS")
@@
 		(descr "Resitance 3 pas")
 		(tags "R")
-		(property "Reference" "D36"
+		(property "Reference" "D33_R"
 			(at 0 -1.63 19)
 			(layer "B.SilkS")
@@
 		(descr "Resitance 3 pas")
 		(tags "R")
-		(property "Reference" "D40"
+		(property "Reference" "D44_R"
 			(at 0 -1.63 358)
 			(layer "B.SilkS")
@@
 		(layer "F.Cu")
 		(at 257.047778 166.62998 47)
-		(property "Reference" "RC1-8"
+		(property "Reference" "K42_R"
 			(at 0 4 47)
 			(layer "B.SilkS")
@@
 		(descr "Resitance 3 pas")
 		(tags "R")
-		(property "Reference" "D45"
+		(property "Reference" "D26_R"
 			(at 0 -1.63 178)
 			(layer "B.SilkS")
@@
 		(layer "F.Cu")
 		(at 275.16882 153.654306 25)
-		(property "Reference" "RC2-8"
+		(property "Reference" "K43_R"
 			(at 0 4 25)
 			(layer "B.SilkS")
@@
 		(layer "F.Cu")
 		(at 288.353025 121.552106 19)
-		(property "Reference" "RC1-7"
+		(property "Reference" "K32_R"
 			(at 0 4 19)
 			(layer "B.SilkS")
@@
 		(descr "Resitance 3 pas")
 		(tags "R")
-		(property "Reference" "D25"
+		(property "Reference" "D21_R"
 			(at 0 -1.63 14)
 			(layer "B.SilkS")
@@
 		(layer "F.Cu")
 		(at 262.007187 93.647539 7.12)
-		(property "Reference" "RC1-5"
+		(property "Reference" "K11_R"
 			(at 0 4 7.12)
 			(layer "B.SilkS")
@@
 		(layer "F.Cu")
 		(at 327.900801 117.25779 21.5)
-		(property "Reference" "RC4-7"
+		(property "Reference" "K34_R"
 			(at 0 4 21.5)
 			(layer "B.SilkS")
@@
 		(descr "Resitance 3 pas")
 		(tags "R")
-		(property "Reference" "D43"
+		(property "Reference" "D45_R"
 			(at 0 -1.63 27.4)
 			(layer "B.SilkS")
@@
 		(layer "F.Cu")
 		(at 360.319035 82.17142 -2)
-		(property "Reference" "RC6-5"
+		(property "Reference" "K26_R"
 			(at 0.238961 4.522996 178)
 			(layer "B.SilkS")
@@
 		(layer "F.Cu")
 		(at 340.633874 89.379195 6)
-		(property "Reference" "RC5-5"
+		(property "Reference" "K25_R"
 			(at 0 4 6)
 			(layer "B.SilkS")
@@
 		(layer "F.Cu")
 		(at 365.304971 103.44885 18.2)
-		(property "Reference" "RC6-6"
+		(property "Reference" "K36_R"
 			(at 0 4 18.2)
 			(layer "B.SilkS")
@@
 		(descr "Resitance 3 pas")
 		(tags "R")
-		(property "Reference" "D39"
-			(at -1.076929 1.922495 21.5)
+		(property "Reference" "D34_R"
+			(at 0.023354 -1.706483 21.5)
 			(layer "B.SilkS")
 			(effects
@@
 		(descr "Resitance 3 pas")
 		(tags "R")
-		(property "Reference" "D41"
+		(property "Reference" "D25_R"
 			(at 0 -1.63 6)
 			(layer "B.SilkS")
@@
 		(descr "Resitance 3 pas")
 		(tags "R")
-		(property "Reference" "D33"
+		(property "Reference" "D43_R"
 			(at 0 -1.63 25)
 			(layer "B.SilkS")
@@
 		(layer "F.Cu")
 		(at 373.828438 122.335777 28.75)
-		(property "Reference" "RC6-7"
+		(property "Reference" "K46_R"
 			(at 0 4 28.75)
 			(layer "B.SilkS")
@@
 		(descr "Resitance 3 pas")
 		(tags "R")
-		(property "Reference" "D35"
+		(property "Reference" "D23_R"
 			(at 0 -1.63 10)
 			(layer "B.SilkS")
@@
 		(layer "F.Cu")
 		(at 355.008317 128.044207 27.4)
-		(property "Reference" "RC5-7"
+		(property "Reference" "K45_R"
 			(at 0 4 27.4)
 			(layer "B.SilkS")
@@
 		(layer "F.Cu")
 		(at 346.164875 109.235615 15.9)
-		(property "Reference" "RC5-6"
+		(property "Reference" "K35_R"
 			(at 0 4 15.9)
 			(layer "B.SilkS")
@@
 		(layer "F.Cu")
 		(at 321.784402 97.810765 13)
-		(property "Reference" "RC4-6"
+		(property "Reference" "K24_R"
 			(at 0 4 13)
 			(layer "B.SilkS")
@@
 		(descr "Resitance 3 pas")
 		(tags "R")
-		(property "Reference" "D30"
+		(property "Reference" "D42_R"
 			(at -0.000001 -1.63 47)
 			(layer "B.SilkS")
@@
 		(descr "Resitance 3 pas")
 		(tags "R")
-		(property "Reference" "D34"
+		(property "Reference" "D13_R"
 			(at 0 -1.63 4.5)
 			(layer "B.SilkS")
@@
 		(descr "Resitance 3 pas")
 		(tags "R")
-		(property "Reference" "D38"
+		(property "Reference" "D24_R"
 			(at 0 -1.63 13)
 			(layer "B.SilkS")
@@
 		(layer "F.Cu")
 		(at 306.053025 113.552106 19)
-		(property "Reference" "RC3-7"
+		(property "Reference" "K33_R"
 			(at 0 4 19)
 			(layer "B.SilkS")
@@
 		(layer "F.Cu")
 		(at 283.083157 101.993178 11.4)
-		(property "Reference" "RC2-6"
+		(property "Reference" "K22_R"
 			(at 0 4 11.4)
 			(layer "B.SilkS")
@@
 		(descr "Resitance 3 pas")
 		(tags "R")
-		(property "Reference" "D37"
+		(property "Reference" "D14_R"
 			(at 0 -1.63 6)
 			(layer "B.SilkS")
@@
 		(descr "Resitance 3 pas")
 		(tags "R")
-		(property "Reference" "D42"
+		(property "Reference" "D35_R"
 			(at -0.000001 -1.63 15.9)
 			(layer "B.SilkS")
@@
 		(layer "F.Cu")
 		(at 301.093671 93.616608 10)
-		(property "Reference" "RC3-6"
+		(property "Reference" "K23_R"
 			(at 0 4 10)
 			(layer "B.SilkS")
@@
 		(layer "F.Cu")
 		(at 383.929905 96.95811 22)
-		(property "Reference" "RC5-8"
+		(property "Reference" "K37_R"
 			(at 0 3.999999 22)
 			(layer "B.SilkS")
@@
 		(descr "Resitance 3 pas")
 		(tags "R")
-		(property "Reference" "D46"
-			(at 0 -1.63 18.2)
+		(property "Reference" "D36_R"
+			(at 0 -1.63 18.199)
 			(layer "B.SilkS")
 			(effects
@@
 		(layer "F.Cu")
 		(at 297.700241 149.285069 -2)
-		(property "Reference" "RC4-8"
+		(property "Reference" "K44_R"
 			(at 0 4 178)
 			(layer "B.SilkS")
@@
 		(descr "Resitance 3 pas")
 		(tags "R")
-		(property "Reference" "D26"
+		(property "Reference" "D31_R"
 			(at 0 -1.63 21)
 			(layer "B.SilkS")
@@
 		(layer "F.Cu")
 		(at 265.847092 113.420359 14)
-		(property "Reference" "RC0-6"
+		(property "Reference" "K21_R"
 			(at 0 4 14)
 			(layer "B.SilkS")
@@
 		(layer "F.Cu")
 		(at 244.677541 184.113216 62)
-		(property "Reference" "RC0-8"
+		(property "Reference" "K41_R"
 			(at 0 4 62)
 			(layer "B.SilkS")
@@
 		(layer "F.Cu")
 		(at 318.633874 77.879195 6)
-		(property "Reference" "RC4-5"
+		(property "Reference" "K14_R"
 			(at 0 4 6)
 			(layer "B.SilkS")
@@
 		(descr "Resitance 3 pas")
 		(tags "R")
-		(property "Reference" "D44"
+		(property "Reference" "D37_R"
 			(at 0 -1.63 22)
 			(layer "B.SilkS")
@@
 		(descr "Resitance 3 pas")
 		(tags "R")
-		(property "Reference" "D29"
+		(property "Reference" "D32_R"
 			(at 0 -1.63 19)
 			(layer "B.SilkS")
@@
 		(descr "Resitance 3 pas")
 		(tags "R")
-		(property "Reference" "D32"
+		(property "Reference" "D22_R"
 			(at 0 -1.63 11.4)
 			(layer "B.SilkS")
@@
 		(descr "Resitance 3 pas")
 		(tags "R")
-		(property "Reference" "D47"
+		(property "Reference" "D46_R"
 			(at 0 -1.63 28.75)
 			(layer "B.SilkS")
@@
 		(layer "F.Cu")
 		(at 271.871544 132.657198 21)
-		(property "Reference" "RC0-7"
+		(property "Reference" "K31_R"
 			(at 0 4 21)
 			(layer "B.SilkS")
@@
 		(descr "Resitance 3 pas")
 		(tags "R")
-		(property "Reference" "D31"
+		(property "Reference" "D12_R"
 			(at 0 -1.63 5)
 			(layer "B.SilkS")
@@
 		(layer "F.Cu")
 		(at 298.935064 73.74389 4.5)
-		(property "Reference" "RC3-5"
+		(property "Reference" "K13_R"
 			(at 0.000001 4 4.5)
 			(layer "B.SilkS")
@@
 		)
 		(fp_line
-			(start -9.524997 -9.525)
-			(end 9.525 -9.524997)
+			(start -9.524996 -9.525)
+			(end 9.525 -9.524996)
 			(stroke
 				(width 0.15)
@@
 		)
 		(fp_line
-			(start -9.525 9.524997)
-			(end -9.524997 -9.525)
+			(start -9.525 9.524996)
+			(end -9.524996 -9.525)
 			(stroke
 				(width 0.15)
@@
 		)
 		(fp_line
-			(start 9.525 -9.524997)
-			(end 9.524997 9.525)
+			(start 9.525 -9.524996)
+			(end 9.524996 9.525)
 			(stroke
 				(width 0.15)
@@
 		)
 		(fp_line
-			(start 9.524997 9.525)
-			(end -9.525 9.524997)
+			(start 9.524996 9.525)
+			(end -9.525 9.524996)
 			(stroke
 				(width 0.15)

Commit message: feat: finish wire for right
Parts:
- removed D1, D10, D11, D12, D13, D14, D15, D16, D17, D18, D19, D2, D20, D21, D22, D23, D24, D3, D4, D5, D6, D7, D8, D9, DI1, DI2, DI3, DI4, DI5, DI6, DI7, DI8, DS1, DS2, DS3, DS4, DS5, DS6, DS7, DS8: 1N4148, kbd_Parts:Diode_TH_SMD
- removed J9: Conn_01x06, Connector_PinHeader_2.54mm:PinHeader_1x06_P2.54mm_Horizontal
- removed RC0-2, RC0-3, RC0-4, RC1-1, RC1-3, RC1-4, RC2-1, RC2-2, RC2-4, RC3-1, RC3-2, RC3-3, RC4-1, RC4-2, RC4-3, RC4-4, RC5-1, RC5-2, RC5-3, RC5-4, RC6-1, RC6-2, RC6-3, RC6-4: SW_Push, kbd_SW:CherryMX_Hotswap_1u
- added D_L_11: 1N4148, kbd_Parts:Diode_TH_SMD, F.Cu at (86.6, 46.8)
- added D_L_12: 1N4148, kbd_Parts:Diode_TH_SMD, F.Cu at (86.6, 49.4)
- added D_L_13: 1N4148, kbd_Parts:Diode_TH_SMD, F.Cu at (86.6, 52.1)
- added D_L_14: 1N4148, kbd_Parts:Diode_TH_SMD, F.Cu at (86.6, 54.7)
- added D_L_21: 1N4148, kbd_Parts:Diode_TH_SMD, F.Cu at (86.6, 57.4)
- added D_L_22: 1N4148, kbd_Parts:Diode_TH_SMD, F.Cu at (86.6, 60.0)
- added D_L_23: 1N4148, kbd_Parts:Diode_TH_SMD, F.Cu at (86.6, 62.7)
- added D_L_24: 1N4148, kbd_Parts:Diode_TH_SMD, F.Cu at (86.6, 65.3)
- added D_L_25: 1N4148, kbd_Parts:Diode_TH_SMD, F.Cu at (96.7, 46.8)
- added D_L_26: 1N4148, kbd_Parts:Diode_TH_SMD, F.Cu at (96.7, 49.4)
- added D_L_31: 1N4148, kbd_Parts:Diode_TH_SMD, F.Cu at (96.7, 52.1)
- added D_L_32: 1N4148, kbd_Parts:Diode_TH_SMD, F.Cu at (96.7, 54.7)
- added D_L_33: 1N4148, kbd_Parts:Diode_TH_SMD, F.Cu at (96.7, 57.4)
- added D_L_34: 1N4148, kbd_Parts:Diode_TH_SMD, F.Cu at (96.7, 60.0)
- added D_L_35: 1N4148, kbd_Parts:Diode_TH_SMD, F.Cu at (96.7, 62.7)
- added D_L_36: 1N4148, kbd_Parts:Diode_TH_SMD, F.Cu at (96.7, 65.3)
- added D_L_37: 1N4148, kbd_Parts:Diode_TH_SMD, F.Cu at (106.7, 46.8)
- added D_L_41: 1N4148, kbd_Parts:Diode_TH_SMD, F.Cu at (106.7, 49.4)
- added D_L_42: 1N4148, kbd_Parts:Diode_TH_SMD, F.Cu at (106.7, 52.1)
- added D_L_43: 1N4148, kbd_Parts:Diode_TH_SMD, F.Cu at (106.7, 54.7)
- added D_L_44: 1N4148, kbd_Parts:Diode_TH_SMD, F.Cu at (106.7, 57.4)
- added D_L_45: 1N4148, kbd_Parts:Diode_TH_SMD, F.Cu at (106.7, 60.0)
- added D_L_46: 1N4148, kbd_Parts:Diode_TH_SMD, F.Cu at (106.7, 62.7)
- added K_L_11: SW_Push, kbd_SW:CherryMX_Hotswap_1u, F.Cu at (37.5, 52.6)
- added K_L_12: SW_Push, kbd_SW:CherryMX_Hotswap_1u, F.Cu at (37.5, 62.3)
- added K_L_13: SW_Push, kbd_SW:CherryMX_Hotswap_1u, F.Cu at (37.5, 72.0)
- added K_L_14: SW_Push, kbd_SW:CherryMX_Hotswap_1u, F.Cu at (37.5, 81.7)
- added K_L_21: SW_Push, kbd_SW:CherryMX_Hotswap_1u, F.Cu at (37.5, 91.3)
- added K_L_22: SW_Push, kbd_SW:CherryMX_Hotswap_1u, F.Cu at (37.5, 101.0)
- added K_L_23: SW_Push, kbd_SW:CherryMX_Hotswap_1u, F.Cu at (37.5, 110.7)
- added K_L_24: SW_Push, kbd_SW:CherryMX_Hotswap_1u, F.Cu at (37.5, 120.4)
- added K_L_25: SW_Push, kbd_SW:CherryMX_Hotswap_1u, F.Cu at (55.4, 52.6)
- added K_L_26: SW_Push, kbd_SW:CherryMX_Hotswap_1u, F.Cu at (55.4, 62.3)
- added K_L_31: SW_Push, kbd_SW:CherryMX_Hotswap_1u, F.Cu at (55.4, 72.0)
- added K_L_32: SW_Push, kbd_SW:CherryMX_Hotswap_1u, F.Cu at (55.4, 81.7)
- added K_L_33: SW_Push, kbd_SW:CherryMX_Hotswap_1u, F.Cu at (55.4, 91.3)
- added K_L_34: SW_Push, kbd_SW:CherryMX_Hotswap_1u, F.Cu at (55.4, 101.0)
- added K_L_35: SW_Push, kbd_SW:CherryMX_Hotswap_1u, F.Cu at (55.4, 110.7)
- added K_L_36: SW_Push, kbd_SW:CherryMX_Hotswap_1u, F.Cu at (55.4, 120.4)
- added K_L_37: SW_Push, kbd_SW:CherryMX_Hotswap_1u, F.Cu at (73.3, 52.6)
- added K_L_41: SW_Push, kbd_SW:CherryMX_Hotswap_1u, F.Cu at (73.3, 62.3)
- added K_L_42: SW_Push, kbd_SW:CherryMX_Hotswap_1u, F.Cu at (73.3, 72.0)
- added K_L_43: SW_Push, kbd_SW:CherryMX_Hotswap_1u, F.Cu at (73.3, 81.7)
- added K_L_44: SW_Push, kbd_SW:CherryMX_Hotswap_1u, F.Cu at (73.3, 91.3)
- added K_L_45: SW_Push, kbd_SW:CherryMX_Hotswap_1u, F.Cu at (73.3, 101.0)
- added K_L_46: SW_Push, kbd_SW:CherryMX_Hotswap_1u, F.Cu at (73.3, 110.7)
- R3, R4: moved to B.Cu
- moved C4 97.0 mm to (228.9, 130.0), turned to 90 degrees
- moved R4 93.9 mm to (229.1, 139.7), turned to 90 degrees
- moved SW4 89.9 mm to (243.3, 140.6), turned to 0 degrees
- moved C3 86.6 mm to (236.7, 127.6), turned to -90 degrees
- moved R3 82.6 mm to (232.6, 134.2), turned to 90 degrees
- moved J7 81.3 mm to (235.0, 155.6), turned to 180 degrees
- renumbered D11_R to D_R_11, D12_R to D_R_12, D13_R to D_R_13, D14_R to D_R_14, D21_R to D_R_21, D22_R to D_R_22, D23_R to D_R_23, D24_R to D_R_24, D25_R to D_R_25, D26_R to D_R_26, D31_R to D_R_31, D32_R to D_R_32, D33_R to D_R_33, D34_R to D_R_34, D35_R to D_R_35, D36_R to D_R_36, D37_R to D_R_37, D41_R to D_R_41, D42_R to D_R_42, D43_R to D_R_43, D44_R to D_R_44, D45_R to D_R_45, D46_R to D_R_46, K11_R to K_R_11, K12_R to K_R_12, K13_R to K_R_13, K14_R to K_R_14, K21_R to K_R_21, K22_R to K_R_22, K23_R to K_R_23, K24_R to K_R_24, K25_R to K_R_25, K26_R to K_R_26, K31_R to K_R_31, K32_R to K_R_32, K33_R to K_R_33, K34_R to K_R_34, K35_R to K_R_35, K36_R to K_R_36, K37_R to K_R_37, K41_R to K_R_41, K42_R to K_R_42, K43_R to K_R_43, K44_R to K_R_44, K45_R to K_R_45, K46_R to K_R_46
Connections:
- D_R_11 pad 1: Net-(D28-K) -> Row1_R
- D_R_12 pad 1: Net-(D28-K) -> Row1_R
- D_R_13 pad 1: Net-(D28-K) -> Row1_R
- D_R_14 pad 1: Net-(D28-K) -> Row1_R
- D_R_21 pad 1: Net-(D25-K) -> Row2_R
- D_R_22 pad 1: Net-(D25-K) -> Row2_R
- D_R_23 pad 1: Net-(D25-K) -> Row2_R
- D_R_24 pad 1: Net-(D25-K) -> Row2_R
- D_R_25 pad 1: Net-(D28-K) -> Row2_R
- D_R_26 pad 1: Net-(D28-K) -> Row2_R
- D_R_31 pad 1: Net-(D26-K) -> Row3_R
- D_R_32 pad 1: Net-(D26-K) -> Row3_R
- D_R_33 pad 1: Net-(D26-K) -> Row3_R
- D_R_34 pad 1: Net-(D26-K) -> Row3_R
- D_R_35 pad 1: Net-(D25-K) -> Row3_R
- D_R_36 pad 1: Net-(D25-K) -> Row3_R
- D_R_37 pad 1: Net-(D27-K) -> Row3_R
- D_R_41 pad 1: Net-(D27-K) -> Row4_R
- D_R_42 pad 1: Net-(D27-K) -> Row4_R
- D_R_43 pad 1: Net-(D27-K) -> Row4_R
- D_R_44 pad 1: Net-(D27-K) -> Row4_R
- D_R_45 pad 1: Net-(D26-K) -> Row4_R
- D_R_46 pad 1: Net-(D26-K) -> Row4_R
- K_R_11 pad 1: Key1_R -> Col1_R
- K_R_12 pad 1: Key2_R -> Col2_R
- K_R_13 pad 1: Key3_R -> Col3_R
- K_R_14 pad 1: Key4_R -> Col4_R
- K_R_21 pad 1: Key0_R -> Col1_R
- K_R_22 pad 1: Key2_R -> Col2_R
- K_R_23 pad 1: Key3_R -> Col3_R
- K_R_24 pad 1: Key4_R -> Col4_R
- K_R_25 pad 1: Key5_R -> Col5_R
- K_R_26 pad 1: Key6_R -> Col6_R
- K_R_31 pad 1: Key0_R -> Col1_R
- K_R_32 pad 1: Key1_R -> Col2_R
- K_R_33 pad 1: Key3_R -> Col3_R
- K_R_34 pad 1: Key4_R -> Col4_R
- K_R_35 pad 1: Key5_R -> Col5_R
- K_R_36 pad 1: Key6_R -> Col6_R
- K_R_37 pad 1: Key5_R -> Col7_R
- K_R_41 pad 1: Key0_R -> Col1_R
- K_R_42 pad 1: Key1_R -> Col2_R
- K_R_43 pad 1: Key2_R -> Col3_R
- K_R_44 pad 1: Key4_R -> Col4_R
- K_R_45 pad 1: Key5_R -> Col5_R
- K_R_46 pad 1: Key6_R -> Col6_R
- U1 pad 14: GND -> GND_L
- U1 pad 17: Key0_L -> Col1_L
- U1 pad 18: Key1_L -> Col2_L
- U1 pad 19: Key2_L -> Col3_L
- U1 pad 20: Key3_L -> Col4_L
- U1 pad 21: Key4_L -> Col5_L
- U1 pad 22: Key5_L -> Col6_L
- U1 pad 23: Key6_L -> Col7_L
- U1 pad 24: KeyINT_L -> Row1_L
- U1 pad 25: unconnected-(U1-P1.01-LF-Pad25) -> Row4_L
- U1 pad 26: unconnected-(U1-P1.02-LF-Pad26) -> Row3_L
- U1 pad 27: unconnected-(U1-P1.07-LF-Pad27) -> Row2_L
- U1 pad 5: SCLK_L -> unconnected-(U1-P0.17-Pad5)
- U1 pad 6: MISO_L -> unconnected-(U1-P0.20-Pad6)
- U1 pad 7: MOSI_L -> unconnected-(U1-P0.22-Pad7)
- U1 pad 8: CS_L -> unconnected-(U1-P0.24-Pad8)
- U2 pad 17: Key0_R -> Col1_R
- U2 pad 18: Key1_R -> Col2_R
- U2 pad 19: Key2_R -> Col3_R
- U2 pad 20: Key3_R -> Col4_R
- U2 pad 21: Key4_R -> Col5_R
- U2 pad 22: Key5_R -> Col6_R
- U2 pad 23: Key6_R -> Col7_R
- U2 pad 24: KeyINT_R -> Row1_R
- U2 pad 25: unconnected-(U2-P1.01-LF-Pad25) -> Row4_R
- U2 pad 26: unconnected-(U2-P1.02-LF-Pad26) -> Row3_R
- U2 pad 27: unconnected-(U2-P1.07-LF-Pad27) -> Row2_R
- U2 pad 5: SCLK_R -> unconnected-(U2-P0.17-Pad5)
- U2 pad 6: MISO_R -> unconnected-(U2-P0.20-Pad6)
- U2 pad 7: MOSI_R -> unconnected-(U2-P0.22-Pad7)
- U2 pad 8: CS_R -> unconnected-(U2-P0.24-Pad8)
Routing:
- net Row4_R: track 0.00 -> 234.2 mm
- net Net-(D27-K): track 231.5 -> 0.00 mm, vias 2 -> 0
- net Key5_R: track 210.1 -> 0.00 mm, vias 6 -> 0
- net Col6_R: track 0.00 -> 206.5 mm, vias 0 -> 1
- net Col7_R: track 0.00 -> 200.1 mm, vias 0 -> 1
- net Row3_R: track 0.00 -> 195.0 mm
- net Col4_R: track 0.00 -> 193.4 mm, vias 0 -> 1
- net Col5_R: track 0.00 -> 188.9 mm, vias 0 -> 1
- net Net-(D26-K): track 181.0 -> 0.00 mm
- net Col3_R: track 0.00 -> 179.3 mm, vias 0 -> 1
- net Net-(D28-K): track 178.4 -> 0.00 mm, vias 3 -> 0
- net Net-(D25-K): track 173.6 -> 0.00 mm
- net Key4_R: track 162.4 -> 0.00 mm, vias 3 -> 0
- net Key6_R: track 161.6 -> 0.00 mm, vias 2 -> 0
- net Col2_R: track 0.00 -> 156.9 mm, vias 0 -> 1
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