File: ErgoNexus.kicad_sch (KiCad schematic)
At the start: 110 parts, among them J7 Conn_01x02, J8 Conn_01x02, SW1 SW_Push, SW3 SW_Push, U1 SuperMini nRF52840, U2 SuperMini nRF52840

Commit message: fix: キーソケットをGatronLP(KS-33B)用に変更
Parts:
- K_L_11, K_L_12, K_L_13, K_L_14, K_L_15, K_L_16, K_L_21, K_L_22, K_L_23, K_L_24, K_L_25, K_L_26, K_L_31, K_L_32, K_L_33, K_L_34, K_L_35, K_L_36, K_L_41, K_L_42, K_L_43, K_L_44, K_R_11, K_R_12, K_R_13, K_R_14, K_R_15, K_R_16, K_R_21, K_R_22, K_R_23, K_R_24, K_R_25, K_R_26, K_R_31, K_R_32, K_R_33, K_R_34, K_R_35, K_R_36, K_R_41, K_R_42, K_R_43, K_R_44: footprint kbd_SW:CherryMX_Hotswap_1u -> mystster:GatronLP_Hotswap_1u
Changed lines of the file:
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@@
 			)
 		)
-		(property "Footprint" "kbd_SW:CherryMX_Hotswap_1u"
+		(property "Footprint" "mystster:GatronLP_Hotswap_1u"
 			(at 63.5 107.95 0)
 			(hide yes)
@@
 			)
 		)
-		(property "Footprint" "kbd_SW:CherryMX_Hotswap_1u"
+		(property "Footprint" "mystster:GatronLP_Hotswap_1u"
 			(at 81.28 107.95 0)
 			(hide yes)
@@
 			)
 		)
-		(property "Footprint" "kbd_SW:CherryMX_Hotswap_1u"
+		(property "Footprint" "mystster:GatronLP_Hotswap_1u"
 			(at 237.49 135.89 0)
 			(hide yes)
@@
 			)
 		)
-		(property "Footprint" "kbd_SW:CherryMX_Hotswap_1u"
+		(property "Footprint" "mystster:GatronLP_Hotswap_1u"
 			(at 166.37 107.95 0)
 			(hide yes)
@@
 			)
 		)
-		(property "Footprint" "kbd_SW:CherryMX_Hotswap_1u"
+		(property "Footprint" "mystster:GatronLP_Hotswap_1u"
 			(at 184.15 135.89 0)
 			(hide yes)
@@
 			)
 		)
-		(property "Footprint" "kbd_SW:CherryMX_Hotswap_1u"
+		(property "Footprint" "mystster:GatronLP_Hotswap_1u"
 			(at 255.27 121.92 0)
 			(hide yes)
@@
 			)
 		)
-		(property "Footprint" "kbd_SW:CherryMX_Hotswap_1u"
+		(property "Footprint" "mystster:GatronLP_Hotswap_1u"
 			(at 134.62 121.92 0)
 			(hide yes)
@@
 			)
 		)
-		(property "Footprint" "kbd_SW:CherryMX_Hotswap_1u"
+		(property "Footprint" "mystster:GatronLP_Hotswap_1u"
 			(at 99.06 149.86 0)
 			(hide yes)
@@
 			)
 		)
-		(property "Footprint" "kbd_SW:CherryMX_Hotswap_1u"
+		(property "Footprint" "mystster:GatronLP_Hotswap_1u"
 			(at 99.06 135.89 0)
 			(hide yes)
@@
 			)
 		)
-		(property "Footprint" "kbd_SW:CherryMX_Hotswap_1u"
+		(property "Footprint" "mystster:GatronLP_Hotswap_1u"
 			(at 184.15 107.95 0)
 			(hide yes)
@@
 			)
 		)
-		(property "Footprint" "kbd_SW:CherryMX_Hotswap_1u"
+		(property "Footprint" "mystster:GatronLP_Hotswap_1u"
 			(at 219.71 135.89 0)
 			(hide yes)
@@
 			)
 		)
-		(property "Footprint" "kbd_SW:CherryMX_Hotswap_1u"
+		(property "Footprint" "mystster:GatronLP_Hotswap_1u"
 			(at 184.15 121.92 0)
 			(hide yes)
@@
 			)
 		)
-		(property "Footprint" "kbd_SW:CherryMX_Hotswap_1u"
+		(property "Footprint" "mystster:GatronLP_Hotswap_1u"
 			(at 201.93 149.86 0)
 			(hide yes)
@@
 			)
 		)
-		(property "Footprint" "kbd_SW:CherryMX_Hotswap_1u"
+		(property "Footprint" "mystster:GatronLP_Hotswap_1u"
 			(at 45.72 135.89 0)
 			(hide yes)
@@
 			)
 		)
-		(property "Footprint" "kbd_SW:CherryMX_Hotswap_1u"
+		(property "Footprint" "mystster:GatronLP_Hotswap_1u"
 			(at 116.84 121.92 0)
 			(hide yes)
@@
 			)
 		)
-		(property "Footprint" "kbd_SW:CherryMX_Hotswap_1u"
+		(property "Footprint" "mystster:GatronLP_Hotswap_1u"
 			(at 201.93 135.89 0)
 			(hide yes)
@@
 			)
 		)
-		(property "Footprint" "kbd_SW:CherryMX_Hotswap_1u"
+		(property "Footprint" "mystster:GatronLP_Hotswap_1u"
 			(at 237.49 107.95 0)
 			(hide yes)
@@
 			)
 		)
-		(property "Footprint" "kbd_SW:CherryMX_Hotswap_1u"
+		(property "Footprint" "mystster:GatronLP_Hotswap_1u"
 			(at 116.84 135.89 0)
 			(hide yes)
@@
 			)
 		)
-		(property "Footprint" "kbd_SW:CherryMX_Hotswap_1u"
+		(property "Footprint" "mystster:GatronLP_Hotswap_1u"
 			(at 45.72 107.95 0)
 			(hide yes)
@@
 			)
 		)
-		(property "Footprint" "kbd_SW:CherryMX_Hotswap_1u"
+		(property "Footprint" "mystster:GatronLP_Hotswap_1u"
 			(at 81.28 149.86 0)
 			(hide yes)
@@
 			)
 		)
-		(property "Footprint" "kbd_SW:CherryMX_Hotswap_1u"
+		(property "Footprint" "mystster:GatronLP_Hotswap_1u"
 			(at 219.71 149.86 0)
 			(hide yes)
@@
 			)
 		)
-		(property "Footprint" "kbd_SW:CherryMX_Hotswap_1u"
+		(property "Footprint" "mystster:GatronLP_Hotswap_1u"
 			(at 184.15 149.86 0)
 			(hide yes)
@@
 			)
 		)
-		(property "Footprint" "kbd_SW:CherryMX_Hotswap_1u"
+		(property "Footprint" "mystster:GatronLP_Hotswap_1u"
 			(at 63.5 121.92 0)
 			(hide yes)
@@
 			)
 		)
-		(property "Footprint" "kbd_SW:CherryMX_Hotswap_1u"
+		(property "Footprint" "mystster:GatronLP_Hotswap_1u"
 			(at 237.49 121.92 0)
 			(hide yes)
@@
 			)
 		)
-		(property "Footprint" "kbd_SW:CherryMX_Hotswap_1u"
+		(property "Footprint" "mystster:GatronLP_Hotswap_1u"
 			(at 45.72 121.92 0)
 			(hide yes)
@@
 			)
 		)
-		(property "Footprint" "kbd_SW:CherryMX_Hotswap_1u"
+		(property "Footprint" "mystster:GatronLP_Hotswap_1u"
 			(at 116.84 149.86 0)
 			(hide yes)
@@
 			)
 		)
-		(property "Footprint" "kbd_SW:CherryMX_Hotswap_1u"
+		(property "Footprint" "mystster:GatronLP_Hotswap_1u"
 			(at 134.62 135.89 0)
 			(hide yes)
@@
 			)
 		)
-		(property "Footprint" "kbd_SW:CherryMX_Hotswap_1u"
+		(property "Footprint" "mystster:GatronLP_Hotswap_1u"
 			(at 99.06 107.95 0)
 			(hide yes)
@@
 			)
 		)
-		(property "Footprint" "kbd_SW:CherryMX_Hotswap_1u"
+		(property "Footprint" "mystster:GatronLP_Hotswap_1u"
 			(at 116.84 107.95 0)
 			(hide yes)
@@
 			)
 		)
-		(property "Footprint" "kbd_SW:CherryMX_Hotswap_1u"
+		(property "Footprint" "mystster:GatronLP_Hotswap_1u"
 			(at 219.71 121.92 0)
 			(hide yes)
@@
 			)
 		)
-		(property "Footprint" "kbd_SW:CherryMX_Hotswap_1u"
+		(property "Footprint" "mystster:GatronLP_Hotswap_1u"
 			(at 81.28 135.89 0)
 			(hide yes)
@@
 			)
 		)
-		(property "Footprint" "kbd_SW:CherryMX_Hotswap_1u"
+		(property "Footprint" "mystster:GatronLP_Hotswap_1u"
 			(at 219.71 107.95 0)
 			(hide yes)
@@
 			)
 		)
-		(property "Footprint" "kbd_SW:CherryMX_Hotswap_1u"
+		(property "Footprint" "mystster:GatronLP_Hotswap_1u"
 			(at 166.37 135.89 0)
 			(hide yes)
@@
 			)
 		)
-		(property "Footprint" "kbd_SW:CherryMX_Hotswap_1u"
+		(property "Footprint" "mystster:GatronLP_Hotswap_1u"
 			(at 201.93 121.92 0)
 			(hide yes)
@@
 			)
 		)
-		(property "Footprint" "kbd_SW:CherryMX_Hotswap_1u"
+		(property "Footprint" "mystster:GatronLP_Hotswap_1u"
 			(at 166.37 121.92 0)
 			(hide yes)
@@
 			)
 		)
-		(property "Footprint" "kbd_SW:CherryMX_Hotswap_1u"
+		(property "Footprint" "mystster:GatronLP_Hotswap_1u"
 			(at 255.27 107.95 0)
 			(hide yes)
@@
 			)
 		)
-		(property "Footprint" "kbd_SW:CherryMX_Hotswap_1u"
+		(property "Footprint" "mystster:GatronLP_Hotswap_1u"
 			(at 255.27 135.89 0)
 			(hide yes)
@@
 			)
 		)
-		(property "Footprint" "kbd_SW:CherryMX_Hotswap_1u"
+		(property "Footprint" "mystster:GatronLP_Hotswap_1u"
 			(at 166.37 149.86 0)
 			(hide yes)
@@
 			)
 		)
-		(property "Footprint" "kbd_SW:CherryMX_Hotswap_1u"
+		(property "Footprint" "mystster:GatronLP_Hotswap_1u"
 			(at 134.62 107.95 0)
 			(hide yes)
@@
 			)
 		)
-		(property "Footprint" "kbd_SW:CherryMX_Hotswap_1u"
+		(property "Footprint" "mystster:GatronLP_Hotswap_1u"
 			(at 134.62 149.86 0)
 			(hide yes)
@@
 			)
 		)
-		(property "Footprint" "kbd_SW:CherryMX_Hotswap_1u"
+		(property "Footprint" "mystster:GatronLP_Hotswap_1u"
 			(at 99.06 121.92 0)
 			(hide yes)
@@
 			)
 		)
-		(property "Footprint" "kbd_SW:CherryMX_Hotswap_1u"
+		(property "Footprint" "mystster:GatronLP_Hotswap_1u"
 			(at 201.93 107.95 0)
 			(hide yes)
@@
 			)
 		)
-		(property "Footprint" "kbd_SW:CherryMX_Hotswap_1u"
+		(property "Footprint" "mystster:GatronLP_Hotswap_1u"
 			(at 81.28 121.92 0)
 			(hide yes)
@@
 			)
 		)
-		(property "Footprint" "kbd_SW:CherryMX_Hotswap_1u"
+		(property "Footprint" "mystster:GatronLP_Hotswap_1u"
 			(at 63.5 135.89 0)
 			(hide yes)

Commit message: feat: 水平ロータリーエンコーダのスイッチ部品を変更
元々の11mmだと高すぎるのでエンコーダを7mmに変更。
それに伴い、switchも高さの低いものに変更する必要があり、フットプリントを変更
Parts:
- RE2, RE4: footprint THQWGD001:THQWGD001C [4pin] #1 -> THQWGD001:THQWGD001C [2pin] #1
Changed lines of the file:
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@@
 			)
 		)
-		(property "Footprint" "THQWGD001:THQWGD001C [4pin] #1"
+		(property "Footprint" "THQWGD001:THQWGD001C [2pin] #1"
 			(at 175.006 73.406 0)
 			(hide yes)
@@
 			)
 		)
-		(property "Footprint" "THQWGD001:THQWGD001C [4pin] #1"
+		(property "Footprint" "THQWGD001:THQWGD001C [2pin] #1"
 			(at 67.056 69.596 0)
 			(hide yes)

Commit message: feat: 水平ロータリーエンコーダの向きを変更
Parts:
- RE2, RE4: footprint THQWGD001:THQWGD001C [2pin] #1 -> THQWGD001:THQWGD001C [2pin] #2
- RE3: value RotaryEncoder_Switch -> RotaryEncoder
Changed lines of the file:
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@@
 			)
 		)
-		(property "Value" "RotaryEncoder_Switch"
+		(property "Value" "RotaryEncoder"
 			(at 235.712 45.212 0)
 			(show_name no)
@@
 			)
 		)
-		(property "Footprint" "THQWGD001:THQWGD001C [2pin] #1"
+		(property "Footprint" "THQWGD001:THQWGD001C [2pin] #2"
 			(at 175.006 73.406 0)
 			(hide yes)
@@
 			)
 		)
-		(property "Footprint" "THQWGD001:THQWGD001C [2pin] #1"
+		(property "Footprint" "THQWGD001:THQWGD001C [2pin] #2"
 			(at 67.056 69.596 0)
 			(hide yes)

Commit message: feat: add assembly info and fix diode footprint
Parts:
- D_L_11, D_L_12, D_L_13, D_L_14, D_L_15, D_L_16, D_L_21, D_L_22, D_L_23, D_L_24, D_L_25, D_L_26, D_L_31, D_L_32, D_L_33, D_L_34, D_L_35, D_L_36, D_L_41, D_L_42, D_L_43, D_L_44, D_L_45, D_L_46, D_R_11, D_R_12, D_R_13, D_R_14, D_R_15, D_R_16, D_R_21, D_R_22, D_R_23, D_R_24, D_R_25, D_R_26, D_R_31, D_R_32, D_R_33, D_R_34, D_R_35, D_R_36, D_R_41, D_R_42, D_R_43, D_R_44, D_R_45, D_R_46: footprint Diode_SMD:D_0402_1005Metric -> Keebio-Parts:D_SOD-323; LCSC (none) -> C2128
- R10, R6, R7, R9: LCSC (none) -> C4109
- R5, R8: LCSC (none) -> C25890
