File: ErgoNexus_kikit.kicad_pcb (KiCad board)
At the start: 2 copper layers, 342 x 152.5 mm, 270 parts, among them J7 Conn_01x02, J8 Conn_01x02, SW1 SW_Push, SW3 SW_Push, U1 SuperMini nRF52840, U2 SuperMini nRF52840

Commit message: feat: add assembly info and fix diode footprint
Parts:
- D_L_11, D_L_12, D_L_13, D_L_14, D_L_15, D_L_16, D_L_21, D_L_22, D_L_23, D_L_24, D_L_25, D_L_26, D_L_31, D_L_32, D_L_33, D_L_34, D_L_35, D_L_36, D_L_41, D_L_42, D_L_43, D_L_44, D_L_45, D_L_46, D_R_11, D_R_12, D_R_13, D_R_14, D_R_15, D_R_16, D_R_21, D_R_22, D_R_23, D_R_24, D_R_25, D_R_26, D_R_31, D_R_32, D_R_33, D_R_34, D_R_35, D_R_36, D_R_41, D_R_42, D_R_43, D_R_44, D_R_45, D_R_46: footprint Diode_SMD:D_0402_1005Metric -> Keebio-Parts:D_SOD-323
- moved D_L_45 0.64 mm to (188.1, 95.8)
- moved D_R_45 0.30 mm to (224.7, 95.5)
Routing:
- net Board_0-Row4_L: track 150.9 -> 154.6 mm
- net Board_0-Net-(D_L_25-A): track 15.8 -> 12.9 mm
- net Board_0-Col6_R: track 285.2 -> 287.1 mm
- net Board_0-Row4_R: track 155.8 -> 154.0 mm
- net Board_0-Col5_L: track 180.4 -> 181.6 mm
- net Board_0-Row3_R: track 163.9 -> 162.7 mm
- net Board_0-Row2_R: track 133.9 -> 134.9 mm
- net Board_0-Net-(D_R_33-A): track 11.6 -> 12.6 mm
- net Board_0-Net-(D_R_31-A): track 11.6 -> 12.4 mm
- net Board_0-Ro2_B_R: track 82.9 -> 83.6 mm
- net Board_0-Net-(D_R_25-A): track 16.1 -> 15.4 mm
- net Board_0-Net-(D_R_13-A): track 16.5 -> 15.9 mm
- net Board_0-Net-(D_L_13-A): track 14.4 -> 13.9 mm
- net Board_0-Net-(D_L_23-A): track 16.0 -> 15.4 mm
Other:
- board text added: "JLCJLCJLCJLC"
