File: ErgoNexus_kikit.kicad_pcb (KiCad board)
At the start: 2 copper layers, 342 x 152.5 mm, 270 parts, among them J7 Conn_01x02, J8 Conn_01x02, SW1 SW_Push, SW3 SW_Push, U1 SuperMini nRF52840, U2 SuperMini nRF52840

Commit message: fix: remove tooling holes
Parts:
- removed KiKit_FID_B_1, KiKit_FID_B_2, KiKit_FID_B_3, KiKit_FID_B_4, KiKit_FID_T_1, KiKit_FID_T_2, KiKit_FID_T_3, KiKit_FID_T_4: Fiducial, Fiducial
- removed KiKit_TO_1, KiKit_TO_2, KiKit_TO_3, KiKit_TO_4: NPTH, NPTH

Commit message: feat: 端に磁石用の切り込みを追加
Parts:
- removed KiKit_MB_16_6, KiKit_MB_16_7, KiKit_MB_16_8, KiKit_MB_2_6, KiKit_MB_2_7, KiKit_MB_2_8: NPTH, NPTH
- added KiKit_MB_10_9: NPTH, NPTH, F.Cu at (176.1, 38.1)
- added KiKit_MB_12_9: NPTH, NPTH, F.Cu at (250.3, 35.8)
- added KiKit_MB_15_11: NPTH, NPTH, F.Cu at (233.8, 164.5)
- added KiKit_MB_4_11: NPTH, NPTH, F.Cu at (177.4, 164.5)
- added KiKit_MB_5_9: NPTH, NPTH, F.Cu at (310.8, 97.6)
- added KiKit_MB_6_9: NPTH, NPTH, F.Cu at (101.9, 94.4)
- moved KiKit_MB_9_1 19.4 mm to (364.0, 59.3)
- moved KiKit_MB_9_5 19.4 mm to (365.2, 63.3)
- moved KiKit_MB_9_3 19.4 mm to (364.6, 61.3)
- moved KiKit_MB_9_4 19.4 mm to (364.9, 62.3)
- moved KiKit_MB_9_2 19.4 mm to (364.3, 60.3)
- moved KiKit_MB_1_3 15.8 mm to (54.7, 63.4)
- moved KiKit_MB_1_1 15.8 mm to (54.1, 65.3)
- moved KiKit_MB_1_2 15.8 mm to (54.4, 64.3)
- moved KiKit_MB_1_5 15.8 mm to (55.4, 61.4)
- moved KiKit_MB_1_4 15.8 mm to (55.1, 62.4)
- moved KiKit_MB_16_5 13.4 mm to (359.3, 44.3)
- moved KiKit_MB_16_4 13.4 mm to (358.9, 43.3)
- moved KiKit_MB_16_3 13.4 mm to (358.6, 42.3)
- moved KiKit_MB_16_2 13.4 mm to (358.3, 41.3)
- moved KiKit_MB_16_1 13.4 mm to (358.0, 40.3)
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Other:
- outline, holes or cut-outs redrawn
